File: uv_lamp/uv_lamp.kicad_pcb (KiCad board)
At the start: 2 copper layers, 132.1 x 83.8 mm, 178 parts, among them J1 Conn_01x03

Commit message: Grox 152x100mm
Parts:
- moved J1 56.1 mm to (58.4, 73.7)
- moved R20 43.2 mm to (73.7, 148.4)
- moved R1 28.7 mm to (101.6, 52.3)
- moved D1 28.7 mm to (101.6, 61.0)
- moved R16 27.0 mm to (254.0, 52.3)
- moved D151 27.0 mm to (254.0, 61.0)
- moved R2 27.0 mm to (111.8, 52.3)
- moved D11 27.0 mm to (111.8, 61.0)
- moved D2 26.5 mm to (101.6, 72.0)
- moved R15 25.4 mm to (243.8, 52.3)
- moved D141 25.4 mm to (243.8, 61.0)
- moved R3 25.4 mm to (121.9, 52.3)
- moved D21 25.4 mm to (121.9, 61.0)
- moved D12 24.6 mm to (111.8, 72.0)
- moved D3 24.4 mm to (101.6, 83.0)
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Routing:
- net Net-(D11-Pad1): track 5.08 -> 0.00 mm
- net Net-(D1-Pad1): track 5.08 -> 0.00 mm
Other:
- board outline removed

Commit message: Power bars
Parts:
- R20: moved to B.Cu
- moved J1 73.3 mm to (76.2, 144.8)
- moved D111 21.7 mm to (193.0, 53.3)
- moved D112 21.7 mm to (193.1, 64.3)
- moved D113 21.7 mm to (193.1, 75.4)
- moved D115 21.7 mm to (193.1, 97.4)
- moved D116 21.7 mm to (193.1, 108.4)
- moved D118 21.7 mm to (193.1, 130.4)
- moved D119 21.7 mm to (193.1, 141.4)
- moved D120 21.7 mm to (193.0, 152.4)
- moved D121 21.7 mm to (203.2, 53.3)
- moved D130 21.7 mm to (203.2, 152.4)
- moved D62 21.7 mm to (142.3, 64.3)
- moved D63 21.7 mm to (142.3, 75.4)
- moved D65 21.7 mm to (142.3, 97.4)
- moved D66 21.7 mm to (142.3, 108.4)
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Routing:
- net Net-(J1-Pad3): track 0.00 -> 378.3 mm
- net Net-(D10-Pad1): track 0.00 -> 169.0 mm
- net Net-(D21-Pad1): track 0.00 -> 8.47 mm
- net Net-(D11-Pad1): track 0.00 -> 8.47 mm
- net Net-(D97-Pad1): track 0.00 -> 8.47 mm
- net Net-(D96-Pad1): track 0.00 -> 8.47 mm
- net Net-(D95-Pad1): track 0.00 -> 8.47 mm
- net Net-(D94-Pad1): track 0.00 -> 8.47 mm
- net Net-(D93-Pad1): track 0.00 -> 8.47 mm
- net Net-(D92-Pad1): track 0.00 -> 8.47 mm
- net Net-(D7-Pad1): track 0.00 -> 8.47 mm
- net Net-(D69-Pad1): track 0.00 -> 8.47 mm
- net Net-(D67-Pad1): track 0.00 -> 8.47 mm
- net Net-(D66-Pad1): track 0.00 -> 8.47 mm
- net Net-(D65-Pad1): track 0.00 -> 8.47 mm
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- added copper zone on B.Cu, net Net-(D10-Pad1)
- added copper zone on B.Cu, net Net-(J1-Pad3)
Other:
- board outline added: 165.1 x 121.9 mm
